Commit message: [modify]: Verify optimized data
1.增加了一个验证数据一致的节点
2.修改了urdf数据

Signed-off-by: 李剑 <lijian29@xiaomi.com>

File: navigation_bringup/urdf/static_tf.urdf (robot description, URDF)
Before this commit: robot cyberdog, 12 links, 11 joints
Joints:
- joint tf2_node_base_to_camera: origin xyz=0.288824 0.000 0.144322 rpy=0 -0.522 3.142 -> xyz=0.288824 0.000 0.144322 rpy=0 -0.524 0
- joint tf2_node_base_to_lidar: origin xyz=0.179 0 0.0837 rpy=0 0 -3.14159 -> xyz=0.179 0 0.0837 rpy=0 0 0
- joint tf2_node_base_to_tof_left_head: origin xyz=0.259 0.03 0.102 rpy=0 -0.266 0.296 -> xyz=0.259 0.03 0.102 rpy=0.296 -0.266 0
- joint tf2_node_base_to_tof_left_rear: origin xyz=-0.021 0.042 -0.051 rpy=0 0 0.296 -> xyz=-0.021 0.042 -0.051 rpy=0.296 0 0
- joint tf2_node_base_to_tof_right_head: origin xyz=0.259 -0.03 0.102 rpy=0 -0.266 -0.296 -> xyz=0.259 -0.03 0.102 rpy=-0.296 -0.266 0
- joint tf2_node_base_to_tof_right_rear: origin xyz=-0.021 -0.042 -0.051 rpy=0 0 -0.296 -> xyz=-0.021 -0.042 -0.051 rpy=-0.296 0 0
- joint tf2_node_uwb_to_head_uwb: origin xyz=0.17 0 0.164 rpy=3.14159 0 0 -> xyz=0.17 0 0.164 rpy=0 0 3.14159
- joint tf2_node_uwb_to_rear_tof: origin xyz=-0.0235 -0.0845 -0.00325 rpy=-1.5708 0 0 -> xyz=-0.0235 -0.0845 -0.00325 rpy=0 0 -1.5708
- joint tf2_node_uwb_to_rear_uwb: origin xyz=-0.023 0.0845 -0.00325 rpy=1.5708 0 0 -> xyz=-0.023 0.0845 -0.00325 rpy=0 0 1.5708

File: navigation_bringup/urdf/static_tf_map.urdf (robot description, URDF)
Before this commit: robot cyberdog, 3 links, 2 joints
Joints:
- joint tf2_node_map_to_odom: origin xyz=0 0 0 rpy=0 0 -3.14159 -> xyz=0 0 0 rpy=0 0 0
- joint tf2_node_map_to_vodom: origin xyz=0 0 0 rpy=0 0 -3.14159 -> xyz=0 0 0 rpy=0 0 0

Commit message: [Modify]: some repos name

File: navigation_bringup/urdf/static_tf.urdf (robot description, URDF)
Before this commit: robot cyberdog, 12 links, 11 joints
Joints:
- joint tf2_node_base_to_camera: origin xyz=0.288824 0.000 0.144322 rpy=0 -0.524 0 -> xyz=0.26932 0.000 0.11543 rpy=0 0.19 0
